File: Top/top_board.kicad_pcb (KiCad board)
At the start: 2 copper layers, 57.8 x 64.8 mm, 17 parts, among them J1 5V, J2 5V, U1 ESP32_DevKit_V1_DOIT

Commit message: actualizacion de placa y libreria para versio 1.1
Parts:
- removed the I2C3V1 at (193.7, 102.8)
- removed I2C5V2: Conn_01x04_Male, Connector_JST:JST_XA_B04B-XASK-1_1x04_P2.50mm_Vertical
- removed LD2: D_Laser_Photo_NType, Connector_JST:JST_XH_B3B-XH-A_1x03_P2.50mm_Vertical
- removed Supply2: Conn_01x03_Male, Connector_JST:JST_XH_B3B-XH-A_1x03_P2.50mm_Vertical
- added G***: LOGO, Images:Spel25x25, F.Cu at (215.6, 94.0)
- added G***: LOGO, Images:LogoSPEL_12x12mm_positive, B.Cu at (231.1, 58.8)
- added J1: Conn_01x06_Pin, Connector_PinHeader_2.54mm:PinHeader_1x06_P2.54mm_Vertical, F.Cu at (192.6, 97.9)
- added J4: Conn_01x04_Pin, Connector_Molex:Molex_Pico-Lock_504050-0491_1x04-1MP_P1.50mm_Horizontal, B.Cu at (204.5, 59.4)
- added R1: 4k7, Resistor_SMD:R_0805_2012Metric_Pad1.20x1.40mm_HandSolder, B.Cu at (202.1, 78.0)
- added U2: BTS5045-1EJA, Package_SO:Infineon_PG-DSO-8-43, B.Cu at (201.7, 70.5)
- J2: value 5V -> Conn_01x06_Pin; footprint Connector_JST:JST_EH_B2B-EH-A_1x02_P2.50mm_Vertical -> Connector_Molex:Molex_Pico-Lock_504050-0691_1x06-1MP_P1.50mm_Horizontal; moved to B.Cu
- U1: moved to B.Cu
- moved J2 3.87 mm to (199.0, 104.8)
- moved U1 1.20 mm to (222.1, 71.4), turned to 180 degrees
- renumbered H3 to H2, H2 to H3, I2C3V3 to I2C3V1, J1 to J3, JP3 to JP1
Connections:
- J2 pad 1: 5V -> SCL5V
- J2 pad 2: GND -> SDA5V
- LD1 pad 2: Net-(LD1-Pad2) -> Net-(J1-Pin_6)
- LD1 pad 3: Net-(LD1-Pad3) -> Net-(J1-Pin_5)
- U1 pad 8: unconnected-(U1-IO25-Pad8) -> Net-(U1-IO25)
Routing:
- net Net-(J1-Pin_6): track 0.00 -> 78.0 mm
- net Net-(J1-Pin_5): track 0.00 -> 76.2 mm, vias 0 -> 1
- net Net-(LD1-Pad2): track 69.4 -> 0.00 mm
- net Net-(LD1-Pad3): track 66.3 -> 0.00 mm
- net 5V: track 67.0 -> 125.9 mm, vias 0 -> 1
- net Net-(U1-IO25): track 0.00 -> 53.2 mm
- net 3V3: track 81.1 -> 41.9 mm, vias 0 -> 1
- net SDA3V3: track 98.5 -> 62.6 mm
- net SCL3V3: track 104.5 -> 69.6 mm
- net SDA5V: track 17.7 -> 44.3 mm
- net SCL5V: track 18.6 -> 42.9 mm
- net Net-(J4-Pin_1): track 0.00 -> 11.3 mm
- net Net-(J4-Pin_4): track 15.1 -> 17.4 mm
- net Net-(J4-Pin_3): track 14.7 -> 13.2 mm
- net GND: track 1.32 -> 0.00 mm
Other:
- board text added: "Jose Pedreros - 2025 Laser Driver Controller Board V1.1 ISS github.com/Japm-Engineer/LaserDriver_ISS"
- board text added: "LD"
- board text added: "PD"
- board text added: "SCL5V"
- board text added: "SDA5V"
- board text removed: "1"
- board text removed: "2"
- board text removed: "3"
- board text removed: "3V3"
- board text removed: "Laser Controller V7 (TOP)"
- board text removed: "SCL_3V3"
- board text removed: "SCL_5V"
- board text removed: "SDA_3V3"
- board text removed: "SDA_5V"
