File: Top/top_board.kicad_sch (KiCad schematic)
At the start: 17 parts, among them J1 5V, J2 5V, U1 ESP32_DevKit_V1_DOIT

Commit message: actualizacion de placa y libreria para versio 1.1
Parts:
- removed I2C3V1, I2C5V2: Conn_01x04_Male, Connector_JST:JST_XA_B04B-XASK-1_1x04_P2.50mm_Vertical, symbol Connector:Conn_01x04_Male
- removed J2: 5V, Connector_JST:JST_EH_B2B-EH-A_1x02_P2.50mm_Vertical, symbol Connector:Conn_01x02_Male
- removed LD2: D_Laser_Photo_NType, Connector_JST:JST_XH_B3B-XH-A_1x03_P2.50mm_Vertical, symbol Device:D_Laser_Photo_NType
- removed Supply2: Conn_01x03_Male, Connector_JST:JST_XH_B3B-XH-A_1x03_P2.50mm_Vertical, symbol Connector:Conn_01x03_Male
- added J1: Conn_01x06_Pin, Connector_PinHeader_2.54mm:PinHeader_1x06_P2.54mm_Vertical, symbol Connector:Conn_01x06_Pin
- added J2: Conn_01x06_Pin, Connector_Molex:Molex_Pico-Lock_504050-0691_1x06-1MP_P1.50mm_Horizontal, symbol Connector:Conn_01x06_Pin
- added J4: Conn_01x04_Pin, Connector_Molex:Molex_Pico-Lock_504050-0491_1x04-1MP_P1.50mm_Horizontal, symbol Connector:Conn_01x04_Pin
- added R1: 4k7, Resistor_SMD:R_0805_2012Metric_Pad1.20x1.40mm_HandSolder, symbol Device:R
- added U2: BTS5045-1EJA, Package_SO:Infineon_PG-DSO-8-43, symbol Power_Management:BTS5045-1EJA
- renumbered H3 to H2, H2 to H3, I2C3V3 to I2C3V1, J1 to J3, JP3 to JP1
Connections:
- net 5V: now also J1.3 (Pin_3), J2.3 (Pin_3), U2.9 (VS)
- net GND: now also J1.4 (Pin_4), J2.4 (Pin_4), J4.2 (Pin_2), R1.2, U2.1 (GND)
- net SCL5V: now also J1.1 (Pin_1), J2.1 (Pin_1)
- net SDA5V: now also J1.2 (Pin_2), J2.2 (Pin_2)
- net at Supply1.1 (Pin_1): now also J4.3 (Pin_3)
- net at Supply1.3 (Pin_3): now also J4.4 (Pin_4)
- net at LD1.2: now also J1.6 (Pin_6), J2.6 (Pin_6)
- net at LD1.3: now also J1.5 (Pin_5), J2.5 (Pin_5)
- net at U1.8 (IO25): now also R1.1, U2.2 (IN)
- new net: J4.1 (Pin_1), U2.6 (OUT), U2.7 (OUT), U2.8 (OUT)
- no-connect marks 0 -> 25
Other:
- moved on the sheet: LD1, Supply1
